File: KEYS_61/KEYS_61.kicad_pcb (KiCad board)
At the start: 2 copper layers, 124 parts, among them J1 Screw_Terminal_01x08, J2 Screw_Terminal_01x08

Commit message: PCB 布局
Parts:
- removed D10, D11, D12, D13, D14, D15, D16, D17, D18, D19, D20, D21, D22, D23, D25, D26, D27, D29, D30, D31, D33, D34, D35, D36, D37, D38, D39, D40, D41, D42, D43, D44, D45, D46, D47, D48, D49, D53, D54, D60, D61, D7, D8, D9: 1N914WT, Keyboard:CHERRY_MX_DIODE
- removed J1: Screw_Terminal_01x08, Connector_PinHeader_2.54mm:PinHeader_1x08_P2.54mm_Vertical
Routing:
- net /row0: track 449.2 -> 1.62 mm
- net /row4: track 431.7 -> 0.00 mm, vias 1 -> 0
- net /row1: track 428.4 -> 0.00 mm
- net /row5: track 402.8 -> 0.00 mm
- net /row2: track 399.3 -> 1.33 mm, vias 1 -> 0
- net /row3: track 373.3 -> 0.77 mm, vias 3 -> 0
- net /row6: track 359.5 -> 0.00 mm
- net /row7: track 319.2 -> 0.00 mm
- net /col6: track 294.8 -> 0.00 mm, vias 4 -> 1
- net /col7: track 269.2 -> 0.51 mm
- net /col5: track 264.4 -> 0.00 mm, vias 1 -> 0
- net /col4: track 246.4 -> 0.00 mm
- net /col0: track 229.4 -> 0.00 mm, vias 1 -> 0
- net /col3: track 222.5 -> 0.00 mm
- net /col2: track 177.3 -> 0.00 mm
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- removed copper zone on B.Cu, net (none)
- removed copper zone on F.Cu, net (none)

Commit message: PCB 自动布线参考
Routing:
- net /row4: track 0.00 -> 323.7 mm
- net /row0: track 1.62 -> 315.6 mm
- net /row5: track 0.00 -> 310.1 mm
- net /row2: track 1.33 -> 295.9 mm
- net /row1: track 0.00 -> 294.3 mm
- net /row6: track 0.00 -> 271.5 mm
- net /col7: track 0.51 -> 252.1 mm
- net /row7: track 0.00 -> 239.6 mm
- net /col6: track 0.00 -> 229.7 mm
- net /row3: track 0.77 -> 228.5 mm
- net /col0: track 0.00 -> 171.4 mm
- net /col3: track 0.00 -> 86.3 mm
- net /col2: track 0.00 -> 48.7 mm
- net Net-(CTRL_LEFT1-Pad1): track 1.62 -> 12.2 mm
- net Net-(D62-Pad1): track 0.89 -> 6.93 mm
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- added copper zone on B.Cu, net (none)
- added copper zone on F.Cu, net (none)
